File: KICAD/full adder npv/full adder npv.kicad_pcb (KiCad board)
At the start: 2 copper layers, 87 parts, among them J2 Barrel_Jack, SW1 SW_SPDT, SW10 SW_SPDT, SW11 SW_SPDT, SW12 SW_SPDT, SW13 SW_SPDT, SW14 SW_SPDT, SW15 SW_SPDT, SW16 SW_SPDT, SW17 SW_Push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

Commit message: ab
Parts:
- moved R41 57.7 mm to (225.5, 65.5)
- moved U3 38.9 mm to (87.3, 112.6)
- moved U4 38.9 mm to (87.3, 101.8)
- moved J2 32.4 mm to (259.5, 67.8)
- moved D17 26.7 mm to (256.5, 83.0)
- moved D19 26.7 mm to (256.7, 95.4)
- moved D20 26.7 mm to (256.7, 101.5)
- moved D21 26.7 mm to (256.7, 107.6)
- moved D22 26.7 mm to (256.7, 114.0)
- moved R33 26.7 mm to (244.9, 83.5)
- moved R34 26.7 mm to (244.9, 89.0)
- moved R35 26.7 mm to (245.4, 95.5)
- moved R36 26.7 mm to (244.4, 101.5)
- moved R37 26.7 mm to (244.9, 107.0)
- moved R38 26.7 mm to (244.4, 114.0)
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
Commit message: KC
Parts:
- moved SW4 100.6 mm to (211.5, 169.5)
- moved SW5 100.5 mm to (35.5, 169.5)
- moved R10 100.2 mm to (136.0, 151.5), turned to 180 degrees
- moved R24 98.1 mm to (111.5, 60.5)
- moved R11 96.2 mm to (155.4, 140.0)
- moved D7 95.4 mm to (179.9, 130.0)
- moved U1 94.1 mm to (107.4, 115.5), turned to 90 degrees
- moved R31 91.3 mm to (216.0, 48.5)
- moved SW16 91.0 mm to (223.5, 31.5)
- moved D12 89.9 mm to (113.7, 71.0)
- moved R9 88.1 mm to (136.0, 141.0), turned to 180 degrees
- moved SW3 75.5 mm to (161.2, 169.5)
- moved SW6 75.4 mm to (85.8, 169.5)
- moved R2 71.1 mm to (32.9, 142.0)
- moved R4 69.7 mm to (57.9, 151.0)
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
Commit message: zb
Parts:
- moved SW16 15.2 mm to (208.3, 31.0)
- moved SW15 13.6 mm to (184.0, 31.0)
- moved SW14 10.3 mm to (158.7, 31.0)
- moved SW13 6.75 mm to (134.3, 31.0)
- moved SW12 6.00 mm to (109.0, 31.0)
- moved R20 5.56 mm to (57.4, 56.0)
- moved R18 5.54 mm to (36.0, 56.0)
- moved R29 5.16 mm to (194.6, 48.5)
- moved R30 5.11 mm to (194.6, 56.0)
- moved R24 4.70 mm to (110.2, 56.0)
- moved R28 4.66 mm to (163.1, 56.0)
- moved R22 4.58 mm to (88.9, 56.0)
- moved R26 4.12 mm to (141.8, 56.0)
- moved D12 3.65 mm to (111.1, 68.5)
- moved SW11 3.44 mm to (83.7, 31.0)
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Routing:
- net GND: track 0.00 -> 394.2 mm
- net /A0: track 0.00 -> 23.7 mm
- net /B7: track 0.00 -> 22.8 mm
- net /B5: track 0.00 -> 21.4 mm
- net /B3: track 0.00 -> 20.1 mm
- net /B1: track 0.00 -> 19.8 mm
- net /B6: track 0.00 -> 19.8 mm
- net /B4: track 0.00 -> 19.7 mm
- net /B0: track 0.00 -> 19.2 mm
Other:
- board outline added: 252 x 172 mm
